Commit message: asdfasd

File: doris_description/urdf/doris.xacro (robot description, xacro)
@@ -320,5 +320,5 @@
     <parent link="shoulder"/>
     <child link="shoulder_pitch"/>
-    <origin xyz="0.065 0.0 0.065" rpy="0 0 0"/>
+    <origin xyz="0.0645 0.0 0.065" rpy="0 0 0"/>
     <axis xyz="0 0 1"/>
     <limit velocity="6.5" effort="1000" lower="${-pi*0.5}" upper="${pi*0.5}" />
@@ -333,5 +333,5 @@
     </collision>
     <visual>
-      <origin xyz="-0.12 -0.08 0.05" rpy="3.1415 0 1.9"/>
+      <origin xyz="-0.1180 -0.08 0.053" rpy="3.1415 0 1.9"/>
       <geometry>
 	      <mesh filename="package://doris_description/urdf/meshes/shoulderpitch.dae" scale="0.001 0.001 0.001"/>
@@ -351,5 +351,5 @@
     <parent link="shoulder_pitch"/>
     <child link="shoulder_elbow_link_down"/>
-    <origin xyz="-0.015 0.0 -0.095" rpy="0 0 0"/>
+    <origin xyz="-0.01105 0.0 -0.0915" rpy="0 0 0"/>
     <axis xyz="0 1 0"/>
     <dynamics damping="0.7"/>
@@ -381,5 +381,5 @@
     <parent link="shoulder_pitch"/>
     <child link="shoulder_elbow_link_up"/>
-    <origin xyz="-0.015 0.0 -0.04" rpy="0 0 0"/>
+    <origin xyz="-0.01105 0.0 -0.0365" rpy="0 0 0"/>
     <axis xyz="0 1 0"/>
     <dynamics damping="0.7"/>
@@ -423,5 +423,5 @@
     </collision>
     <visual>
-      <origin xyz="0.13 -0.04 -0.14" rpy="0 0 1.5707"/>
+      <origin xyz="0.1265 -0.04 -0.14" rpy="0 0 1.5707"/>
       <geometry>
         <mesh filename="package://doris_description/urdf/meshes/elbow.dae" scale="0.001 0.001 0.001"/>
@@ -441,5 +441,5 @@
     <parent link="elbow"/>
     <child link="elbow_wrist_link_up"/>
-    <origin xyz="0.11 0.0 0.0" rpy="0 0 0"/>
+    <origin xyz="0.1045 0.0 0.0" rpy="0 0 0"/>
     <axis xyz="0 1 0"/>
     <dynamics damping="0.7"/>
@@ -453,5 +453,5 @@
     </collision>
     <visual>
-      <origin xyz="-0.03 -0.0425 0.075" rpy="3.08 0 1.5707"/>
+      <origin xyz="-0.027 -0.0425 0.0715" rpy="3.08 0 1.5707"/>
       <geometry>
         <mesh filename="package://doris_description/urdf/meshes/elbow_wrist.dae" scale="0.001 0.001 0.001"/>
@@ -471,5 +471,5 @@
     <parent link="elbow"/>
     <child link="elbow_wrist_link_down"/>
-    <origin xyz="0.11 0.0 -0.055" rpy="0 0 0"/>
+    <origin xyz="0.1045 0.0 -0.055" rpy="0 0 0"/>
     <axis xyz="0 1 0"/>
     <dynamics damping="0.7"/>
@@ -483,5 +483,5 @@
     </collision>
     <visual>
-      <origin xyz="0.24 -0.0425 -0.07" rpy="-0.06 0 1.5707"/>
+      <origin xyz="0.24 -0.0425 -0.0715" rpy="-0.06 0 1.5707"/>
       <geometry>
         <mesh filename="package://doris_description/urdf/meshes/elbow_wrist.dae" scale="0.001 0.001 0.001"/>
@@ -498,10 +498,15 @@
     </inertial>
   </link>
-  <joint name="hearth_joint" type="continuous">
+  <!-- <joint name="hearth_joint" type="continuous">
     <parent link="elbow_wrist_link_up"/>
     <child link="hearth_link"/>
-    <origin xyz="0.21 0.0 0.0" rpy="0 0 0"/>
-    <axis xyz="0 1 0"/>
-    <dynamics damping="0.7"/>
+    <origin xyz="0.214 0.0 0.0" rpy="0 0 0"/>
+    <axis xyz="0 1 0"/>
+    <dynamics damping="0.7"/>
+  </joint>  -->
+  <joint name="hearth_joint" type="fixed">
+    <parent link="elbow_wrist_link_up"/>
+    <child link="hearth_link"/>
+    <origin xyz="0.215 0.0 0.0" rpy="0 0 0"/>
   </joint>
   <link name="hearth_link">
@@ -525,5 +530,5 @@
     <parent link="hearth_link"/>
     <child link="gripper_pitch"/>
-    <origin xyz="0.02 0.0 -0.02" rpy="0 0 0"/>
+    <origin xyz="0.0225 0.0 -0.024" rpy="0 0 0"/>
     <axis xyz="0 1 0"/>
     <dynamics damping="0.7"/>
@@ -537,5 +542,5 @@
     </collision>
     <visual>
-      <origin xyz="-0.0475 0.0 -0.075" rpy="1.5707 0 0"/>
+      <origin xyz="-0.05 0.0 -0.0725" rpy="1.5707 0 0"/>
       <geometry>
         <mesh filename="package://doris_description/urdf/meshes/base_gripper.dae" scale="0.001 0.001 0.001"/>
@@ -555,5 +560,5 @@
     <parent link="gripper_pitch"/>
     <child link="gripper_yaw"/>
-    <origin xyz="0.0025 0.0 -0.035" rpy="0 0 0"/>
+    <origin xyz="0.0 0.0 -0.03" rpy="0 0 0"/>
     <axis xyz="0 0 1"/>
     <dynamics damping="0.7"/>
@@ -585,5 +590,5 @@
     <parent link="gripper_yaw"/>
     <child link="gripper_roll"/>
-    <origin xyz="0.09 0.0 0.045" rpy="0 0 0"/>
+    <origin xyz="0.09 0.0 0.044" rpy="0 0 0"/>
     <axis xyz="1 0 0"/>
     <dynamics damping="0.7"/>
@@ -597,5 +602,5 @@
     </collision>
     <visual>
-      <origin xyz="-0.0 0.0 -0.015" rpy="1.5707 0 0"/>
+      <origin xyz="-0.0 0.0 -0.0125" rpy="1.5707 0 0"/>
       <geometry>
         <mesh filename="package://doris_description/urdf/meshes/gripper_roll.dae" scale="0.001 0.001 0.001"/>
@@ -732,5 +737,5 @@
     </actuator>
   </transmission>
-  <transmission name="trangripperhearth">
+  <!-- <transmission name="trangripperhearth">
     <type>transmission_interface/SimpleTransmission</type>
     <joint name="hearth_joint">
@@ -741,5 +746,5 @@
       <mechanicalReduction>1</mechanicalReduction>
     </actuator>
-  </transmission>
+  </transmission> -->
   <transmission name="trangripperpitch">
     <type>transmission_interface/SimpleTransmission</type>

Commit message: hahahaahha

File: doris_description/urdf/doris.xacro (robot description, xacro)
@@ -498,16 +498,16 @@
     </inertial>
   </link>
-  <!-- <joint name="hearth_joint" type="continuous">
-    <parent link="elbow_wrist_link_up"/>
-    <child link="hearth_link"/>
-    <origin xyz="0.214 0.0 0.0" rpy="0 0 0"/>
-    <axis xyz="0 1 0"/>
-    <dynamics damping="0.7"/>
-  </joint>  -->
-  <joint name="hearth_joint" type="fixed">
+  <joint name="hearth_joint" type="continuous">
     <parent link="elbow_wrist_link_up"/>
     <child link="hearth_link"/>
     <origin xyz="0.215 0.0 0.0" rpy="0 0 0"/>
-  </joint>
+    <axis xyz="0 1 0"/>
+    <dynamics damping="0.7"/>
+  </joint>
+  <!-- <joint name="hearth_joint" type="fixed">
+    <parent link="elbow_wrist_link_up"/>
+    <child link="hearth_link"/>
+    <origin xyz="0.215 0.0 0.0" rpy="0 0 0"/>
+  </joint>  -->
   <link name="hearth_link">
     <visual>
@@ -737,5 +737,5 @@
     </actuator>
   </transmission>
-  <!-- <transmission name="trangripperhearth">
+  <transmission name="trangripperhearth">
     <type>transmission_interface/SimpleTransmission</type>
     <joint name="hearth_joint">
@@ -746,5 +746,5 @@
       <mechanicalReduction>1</mechanicalReduction>
     </actuator>
-  </transmission> -->
+  </transmission>
   <transmission name="trangripperpitch">
     <type>transmission_interface/SimpleTransmission</type>
